File: i2c_interface_terminator.kicad_pcb (KiCad board)
At the start: 2 copper layers, 15 x 11 mm, 0 parts

Commit message: Moved parts.
Other:
- board text added: "i2c_interface_terminator 09/2017 ver 1.0"
- board text removed: "terminator 2 pair 09/2017 ver 1.0"
Changed lines of the file:
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@@
-(kicad_pcb (version 20170123) (host pcbnew no-vcs-found-33cc7b3~60~ubuntu16.04.1)
+(kicad_pcb (version 20170123) (host pcbnew no-vcs-found-e2d3fce~60~ubuntu16.04.1)
   (general
     (thickness 1.6)
@@
   (gr_line (start 92.5 105.5) (end 107.5 105.5) (angle 90) (layer Edge.Cuts) (width 0.2286))
   (gr_line (start 92.5 94.5) (end 92.5 105.5) (angle 90) (layer Edge.Cuts) (width 0.2286))
-  (gr_text "terminator 2 pair 09/2017 ver 1.0" (at 100 104.5) (layer F.SilkS)
+  (gr_text "i2c_interface_terminator\n09/2017 ver 1.0" (at 100 104.5) (layer F.SilkS)
     (effects (font (size 0.508 0.508) (thickness 0.127)))
   )

Commit message: Finished version 1.0.
Parts:
- added P1: HEADER_02X03_FEMALE_SMD, i2c_interface_terminator:HEADER_02x03_FEMALE_SMD, B.Cu at (109.2, 106.0)
- added R1: 604, i2c_interface_terminator:SM0805, F.Cu at (111.8, 103.5)
- added R2: 120, i2c_interface_terminator:SM0805, F.Cu at (114.8, 106.0)
- added R3: 604, i2c_interface_terminator:SM0805, F.Cu at (111.8, 108.6)
- added R4: 604, i2c_interface_terminator:SM0805, F.Cu at (106.7, 103.5)
- added R5: 120, i2c_interface_terminator:SM0805, F.Cu at (103.6, 106.0)
- added R6: 604, i2c_interface_terminator:SM0805, F.Cu at (106.7, 108.6)
Routing:
- net /DSCLP: track 0.00 -> 7.18 mm, vias 0 -> 1
- net /DSCLM: track 0.00 -> 7.18 mm, vias 0 -> 1
- net /DSDAM: track 0.00 -> 7.18 mm, vias 0 -> 1
- net /DSDAP: track 0.00 -> 7.05 mm, vias 0 -> 1
- net VAA: track 0.00 -> 6.16 mm, vias 0 -> 1
- net GND: track 0.00 -> 5.91 mm, vias 0 -> 1
- added copper zone on B.Cu, net GND
- added copper zone on F.Cu, net VAA
Other:
- board size 15 x 11 mm -> 15.2 x 8.9 mm
- net class Default: trace_width 0.25 -> 0.254
